File: hardware/kicad/phase-4-analog-drive/phase-4-analog-drive.kicad_pcb (KiCad board)
At the start: 2 copper layers, 170 x 120 mm, 4 parts, among them J1 MONITOR_DRIVE, J2 HOST_CTRL, U1 TMUX1108PWR, U2 TS5A3159DBVR

Commit message: Phase 4 wip
Parts:
- J2: footprint Connector_PinHeader_2.54mm:PinHeader_1x06_P2.54mm_Vertical -> Connector_PinHeader_2.54mm:PinHeader_1x07_P2.54mm_Vertical
- U1: value TMUX1108PWR -> SN74LV4066APWR; footprint Package_SO:TSSOP-16_4.4x5mm_P0.65mm -> Package_SO:TSSOP-14_4.4x5mm_P0.65mm
- U2: value TS5A3159DBVR -> SN74LVC1G66DBVR; footprint Package_TO_SOT_SMD:SOT-23-6 -> Package_TO_SOT_SMD:SOT-23-5
Changed lines of the file:
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@@
 (kicad_pcb
-	(version 20260206)
+	(version 20250114)
 	(generator "pcbnew")
 	(generator_version "10.0")
@@
 	(title_block
 		(title "Phase 4 Analog Drive PCB")
-		(rev "A")
+		(rev "E")
 		(company "samsung-jog-api")
-		(comment 1 "Prototype placement for U1 TMUX1108 and U2 TS5A3159")
-		(comment 2 "Generated for KiCad 10")
+		(comment 1 "Board placeholder for fail-safe switched resistor architecture")
+		(comment 2 "Schematic now targets SN74LV4066A and SN74LVC1G66")
 	)
 	(layers
@@
 	(net 3 "KEY_ADC2")
 	(net 4 "KEY_ADC1")
-	(net 5 "ADC2_SEL0")
-	(net 6 "ADC2_SEL1")
-	(net 7 "ADC2_EN")
-	(net 8 "ADC1_CENTER_EN")
-	(footprint "Package_SO:TSSOP-16_4.4x5mm_P0.65mm"
+	(net 5 "ADC2_LEFT_EN")
+	(net 6 "ADC2_RIGHT_EN")
+	(net 7 "ADC2_DOWN_EN")
+	(net 8 "ADC2_UP_EN")
+	(net 9 "ADC1_CENTER_EN")
+	(footprint "Package_SO:TSSOP-14_4.4x5mm_P0.65mm"
 		(layer "F.Cu")
 		(at 100 80)
 		(property "Reference" "U1" (at 0 -4 0) (layer "F.SilkS"))
-		(property "Value" "TMUX1108PWR" (at 0 4 0) (layer "F.Fab"))
+		(property "Value" "SN74LV4066APWR" (at 0 4 0) (layer "F.Fab"))
 	)
-	(footprint "Package_TO_SOT_SMD:SOT-23-6"
+	(footprint "Package_TO_SOT_SMD:SOT-23-5"
 		(layer "F.Cu")
 		(at 100 110)
 		(property "Reference" "U2" (at 0 -3 0) (layer "F.SilkS"))
-		(property "Value" "TS5A3159DBVR" (at 0 3 0) (layer "F.Fab"))
+		(property "Value" "SN74LVC1G66DBVR" (at 0 3 0) (layer "F.Fab"))
 	)
 	(footprint "Connector_PinHeader_2.54mm:PinHeader_1x03_P2.54mm_Vertical"
@@
 		(property "Value" "MONITOR_DRIVE" (at 0 8 0) (layer "F.Fab"))
 	)
-	(footprint "Connector_PinHeader_2.54mm:PinHeader_1x06_P2.54mm_Vertical"
+	(footprint "Connector_PinHeader_2.54mm:PinHeader_1x07_P2.54mm_Vertical"
 		(layer "F.Cu")
 		(at 160 80)
 		(property "Reference" "J2" (at 0 -3 0) (layer "F.SilkS"))
-		(property "Value" "HOST_CTRL" (at 0 16 0) (layer "F.Fab"))
+		(property "Value" "HOST_CTRL" (at 0 18 0) (layer "F.Fab"))
 	)
 	(gr_rect (start 20 30) (end 190 150) (layer "Edge.Cuts") (width 0.1) (fill none))

Commit message: Update phase 4 schema, WIP
Parts:
- added C1: 100n, Capacitor_SMD:C_0603_1608Metric, F.Cu at (39.0, 8.00)
- added C2: 100n, Capacitor_SMD:C_0603_1608Metric, F.Cu at (60.0, 36.0)
- added C3: 1u, Capacitor_SMD:C_0603_1608Metric, F.Cu at (71.0, 31.0)
- added R1: 30k, Resistor_SMD:R_0603_1608Metric, F.Cu at (48.0, 19.6)
- added R10: 100k, Resistor_SMD:R_0603_1608Metric, F.Cu at (63.0, 12.5)
- added R11: 100k, Resistor_SMD:R_0603_1608Metric, F.Cu at (63.0, 10.0)
- added R2: 10k, Resistor_SMD:R_0603_1608Metric, F.Cu at (48.0, 17.3)
- added R3: 3.3k, Resistor_SMD:R_0603_1608Metric, F.Cu at (18.0, 17.0)
- added R4: 22k, Resistor_SMD:R_0603_1608Metric, F.Cu at (18.0, 14.7)
- added R6: 22k, Resistor_SMD:R_0603_1608Metric, F.Cu at (66.0, 31.0)
- added R7: 100k, Resistor_SMD:R_0603_1608Metric, F.Cu at (63.0, 20.2)
- added R8: 100k, Resistor_SMD:R_0603_1608Metric, F.Cu at (63.0, 17.6)
- added R9: 100k, Resistor_SMD:R_0603_1608Metric, F.Cu at (63.0, 15.1)
- U1: value SN74LV4066APWR -> MC74HC4066ADTR2G
- U2: value SN74LVC1G66DBVR -> 74LVC1G66LT05ARCQ
- moved J2 107.1 mm to (79.0, 10.0)
- moved U1 92.7 mm to (33.0, 16.0)
- moved U2 90.4 mm to (56.0, 31.0)
- moved J1 77.8 mm to (6.00, 10.0)
Routing:
- net /GND: track 0.00 -> 449.3 mm
- net /+3V3: track 0.00 -> 92.9 mm
- net /KEY_ADC2_BUS: track 0.00 -> 75.0 mm
- net /ADC2_DOWN_EN: track 0.00 -> 69.4 mm
- net /KEY_ADC1_BUS: track 0.00 -> 68.9 mm
- net /ADC2_RIGHT_EN: track 0.00 -> 64.1 mm
- net /ADC1_CENTER_EN: track 0.00 -> 51.1 mm
- net /ADC2_LEFT_EN: track 0.00 -> 48.6 mm
- net /ADC2_UP_EN: track 0.00 -> 45.9 mm
- net /ADC2_LEFT_SW: track 0.00 -> 15.9 mm
- net /ADC2_RIGHT_SW: track 0.00 -> 13.0 mm
- net /ADC2_DOWN_SW: track 0.00 -> 12.3 mm
- net /ADC1_CENTER_SW: track 0.00 -> 12.0 mm
- net /ADC2_UP_SW: track 0.00 -> 11.3 mm
Other:
- board size 170 x 120 mm -> 85 x 45 mm
- board text added: "CJ791 Jog Analog Drive Rev G"
- board text added: "HOST CTRL"
- board text added: "MONITOR"
- board text removed: "Phase 4 Analog Drive Prototype"
