File: hardware/kicad/phase-3-observation-proto/phase-3-observation-proto.kicad_sch (KiCad schematic)
At the start: 34 parts, among them J1 Input_4pin, J2 Host_8pin, Q1 BC547, Q10 BC547, Q11 BC547, Q12 BC547, Q2 BC547, Q3 BC547, Q4 BC547, Q5 BC547, Q6 BC547, Q7 BC547, Q8 BC547, Q9 BC547, U1 74HC86

Commit message: Fix phase-3-observation-proto schematic: replace net_label with label
KiCad 10 uses (label "NAME" (at ...) ...) not (net_label ...).
All 45 net_label blocks converted to correct label format.
Also fixed invalid UUID characters (g-j → hex) on last 3 instances.

Co-Authored-By: Claude Sonnet 4.6 <noreply@anthropic.com>
Connections:
- net Vref1: now reaches Q2.1 (B)
- net Vref1: now also RL2.1
- net Vref4: now reaches RL5.1
- net Vref4: now also Q12.1 (B), Q8.1 (B)
- net KEY_ADC2_BUF: now reaches Q3.1 (B)
- net KEY_ADC2_BUF: now also J1.2 (Pin_2), Q1.1 (B), Q5.1 (B), Q7.1 (B)
- net Vref2: now reaches Q4.1 (B)
- net Vref2: now also RL3.1
- net GND: now reaches J1.1 (Pin_1)
- net KEY_ADC1_BUF: now reaches J1.3 (Pin_3)
- net KEY_ADC1_BUF: now also Q9.1 (B)
- net KEY_LED_BUF: now reaches J1.4 (Pin_4)
- net KEY_LED_BUF: now also Q11.1 (B)
- net Vref3: now reaches Q10.1 (B)
- net Vref3: now also Q6.1 (B), RL4.1
- net OUT1: now reaches U1.1 (A1)
- net OUT4: now reaches U1.10 (B3)
- net OUT2: now reaches U1.2 (B1)
- net OUT2: now also U1.4 (A2)
- net OUT3: now reaches U1.5 (B2)
- net OUT3: now also U1.9 (A3)
