File: hardware/kicad/phase-7-hdmi-ddc-board/phase-7-hdmi-ddc-board.kicad_sch (KiCad schematic)
At the start: 23 parts, among them J1 HDMI_SOURCE, J2 HDMI_MONITOR, J3 HDMI_BOARD_IF, Q1 2N7002, U1 TCA4307DGKR, U2 PCA9306DCTR, U3 TPS2113APWR

Commit message: Phase 7 WIP
Changed lines of the file:
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@@
 	(wire (pts (xy 142.24 107.62) (xy 149.86 107.62)) (stroke (width 0) (type default)))
 	(wire (pts (xy 35.56 222.25) (xy 50.8 222.25)) (stroke (width 0) (type default)))
-	(wire (pts (xy 35.56 224.79) (xy 50.8 224.79)) (stroke (width 0) (type default)))
 	(wire (pts (xy 35.56 219.71) (xy 50.8 219.71)) (stroke (width 0) (type default)))
 	(wire (pts (xy 35.56 217.17) (xy 50.8 217.17)) (stroke (width 0) (type default)))
@@
 	(label "GND" (at 165.1 198.12 0) (effects (font (size 1.27 1.27)) (justify left bottom)))
 	(label "GND" (at 50.8 222.25 0) (effects (font (size 1.27 1.27)) (justify left bottom)))
-	(no_connect (at 50.8 224.79))
+	(no_connect (at 35.56 224.79))
 	(label "+5V_PI" (at 50.8 219.71 0) (effects (font (size 1.27 1.27)) (justify left bottom)))
 	(label "+3V3_PI" (at 50.8 217.17 0) (effects (font (size 1.27 1.27)) (justify left bottom)))
