File: hardware/kicad/analog-drive/analog-drive.kicad_pcb (KiCad board)
At the start: 2 copper layers, 85 x 45 mm, 17 parts, among them J1 MONITOR_DRIVE, J2 HOST_CTRL, U1 MC74HC4066ADTR2G, U2 74LVC1G66LT05ARCQ

Commit message: Fix JOG up and center resistor values
Parts:
- R4, R6: value 22k -> 22R
Changed lines of the file:
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@@
 		)
 	)
-	(footprint "Resistor_SMD:R_0603_1608Metric" (layer "F.Cu") (at 18 14.7) (property "Reference" "R4" (at 0 -1.43 0) (layer "F.SilkS")) (property "Value" "22k" (at 0 1.43 0) (layer "F.Fab")) (attr smd)
+	(footprint "Resistor_SMD:R_0603_1608Metric" (layer "F.Cu") (at 18 14.7) (property "Reference" "R4" (at 0 -1.43 0) (layer "F.SilkS")) (property "Value" "22R" (at 0 1.43 0) (layer "F.Fab")) (attr smd)
 		(pad "1" smd roundrect (at -0.825 0) (size 0.8 0.95) (layers "F.Cu" "F.Mask" "F.Paste") (roundrect_rratio 0.25) (net 12 "/GND"))
 		(pad "2" smd roundrect (at 0.825 0) (size 0.8 0.95) (layers "F.Cu" "F.Mask" "F.Paste") (roundrect_rratio 0.25) (net 11 "/ADC2_UP_SW"))
@@
 		(model "${KICAD10_3DMODEL_DIR}/Resistor_SMD.3dshapes/R_0603_1608Metric.step" (offset (xyz 0 0 0)) (scale (xyz 1 1 1)) (rotate (xyz 0 0 0)))
 	)
-	(footprint "Resistor_SMD:R_0603_1608Metric" (layer "F.Cu") (at 66 31) (property "Reference" "R6" (at 0 -1.43 0) (layer "F.SilkS")) (property "Value" "22k" (at 0 1.43 0) (layer "F.Fab")) (attr smd)
+	(footprint "Resistor_SMD:R_0603_1608Metric" (layer "F.Cu") (at 66 31) (property "Reference" "R6" (at 0 -1.43 0) (layer "F.SilkS")) (property "Value" "22R" (at 0 1.43 0) (layer "F.Fab")) (attr smd)
 		(pad "1" smd roundrect (at -0.825 0) (size 0.8 0.95) (layers "F.Cu" "F.Mask" "F.Paste") (roundrect_rratio 0.25) (net 12 "/GND"))
 		(pad "2" smd roundrect (at 0.825 0) (size 0.8 0.95) (layers "F.Cu" "F.Mask" "F.Paste") (roundrect_rratio 0.25) (net 3 "/ADC1_CENTER_SW"))
