File: hardware/kicad/controller-board/controller-board.kicad_sch (KiCad schematic)
At the start: 35 parts, among them J1 MONITOR_INPUT, J2 PI_GPIO_HEADER, J3 INTER_BOARD, U1 TLV9064IDR, U2 ADS1015IDGSR, U3 74LVC1G17GW, U4 74LVC1G17GW, U5 MC74HC4066ADR2G, U6 74LVC1G66LT05ARCQ

Commit message: Fix JOG up and center resistor values
Parts:
- R16, R17: value 22k -> 22R
Changed lines of the file:
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@@
 			)
 		)
-		(property "Value" "22k"
+		(property "Value" "22R"
 			(at 389.4460 61.468 90)
 			(show_name no)
@@
 			)
 		)
-		(property "Value" "22k"
+		(property "Value" "22R"
 			(at 397.8280 132.588 90)
 			(show_name no)
